Commit message: fastswitch version of the code. not tested on hardware

File: src/gummi_ee_handshake/xacro/gummi_description_ee.urdf.xacro (robot description, xacro)
@@ -2,64 +2,20 @@
   <!-- j5_Link -->
   <robot>
-  <link
-    name="lowerarm_preroll">
-    <inertial>
-      <origin
-        xyz="0.0478250427975905 -0.000316437232932051 -0.0106413204754627"
-        rpy="0 0 0" />
-      <mass
-        value="0.0606243812523471" />
-      <inertia
-        ixx="2.06454707456843E-05"
-        ixy="-1.4331951640169E-06"
-        ixz="6.63107213803745E-06"
-        iyy="4.53417988250448E-05"
-        iyz="3.42736477119013E-07"
-        izz="4.5142289140086E-05" />
-    </inertial>
-    <visual>
-      <origin
-        xyz="0 0 0"
-        rpy="0 0 0" />
-      <geometry>
-        <mesh
-          filename="package://gummi_base_template/meshes/j5_Link.STL" />
-      </geometry>
-      <material
-        name="">
-        <color
-          rgba="0.792156862745098 0.819607843137255 0.933333333333333 1" />
-      </material>
-    </visual>
-    <collision>
-      <origin
-        xyz="0 0 0"
-        rpy="0 0 0" />
-      <geometry>
-        <mesh
-          filename="package://gummi_base_template/meshes/j5_Link.STL" />
-      </geometry>
-    </collision>
-  </link>
-  <!-- j5 -->
-  <joint
-    name="elbow"
-    type="revolute">
-    <origin
-      xyz="0 0 -0.1898"
-      rpy="0 0 0" />
-    <parent
-      link="upperarm" />
-    <child
-      link="lowerarm_preroll" />
-    <axis
-      xyz="0 -1 0" />
-    <!-- <limit
-      lower="-1.5708"
-      upper="1.5708"
-      effort="0"
-      velocity="0" /> -->
-    <limit effort="0" lower="-0.85" upper="0.65" velocity="1.0"/>
-  </joint>
+    <link name="lowerarm_preroll_d">
+        <visual>
+        <origin xyz="0.084 0 -0.012" rpy="0 0 0" />
+        <geometry>
+          <box size=".02 .05 .05" />
+        </geometry>
+        <material name="not Cyan">
+          <color rgba="1 0.7 0.7 1"/>
+        </material>
+      </visual>
+      </link>
+      <joint name="fastswitch" type="fixed">
+        <origin rpy="0 0 0" xyz="0.00 -0.015 0"/>
+        <parent link="lowerarm_preroll_u"/>
+        <child link="lowerarm_preroll_d"/>
+      </joint>
   <!-- j6_Link -->
   <link
@@ -81,9 +37,8 @@
     <visual>
       <origin
-        xyz="0 0 0"
-        rpy="0 0 0" />
-      <geometry>
-        <mesh
-          filename="package://gummi_base_template/meshes/j6_Link.STL" />
+        xyz="0.09 0 0.01"
+        rpy="0 0 0" />
+      <geometry>
+        <box size=".16 .033 .052" />
       </geometry>
       <material
@@ -95,9 +50,8 @@
     <collision>
       <origin
-        xyz="0 0 0"
-        rpy="0 0 0" />
-      <geometry>
-        <mesh
-          filename="package://gummi_base_template/meshes/j6_Link.STL" />
+        xyz="0.09 0 0.01"
+        rpy="0 0 0" />
+      <geometry>
+        <box size=".16 .033 .052" />
       </geometry>
     </collision>
@@ -111,5 +65,5 @@
       rpy="0 0 0" />
     <parent
-      link="lowerarm_preroll" />
+      link="lowerarm_preroll_d" />
     <child
       link="lowerarm" />
@@ -142,9 +96,8 @@
     <visual>
       <origin
-        xyz="0 0 0"
-        rpy="0 0 0" />
-      <geometry>
-        <mesh
-          filename="package://gummi_base_template/meshes/j7_Link.STL" />
+        xyz="0.073 0 0"
+        rpy="0 0 0" />
+      <geometry>
+        <box size=".146 .06 .015" />
       </geometry>
       <material
@@ -156,9 +109,8 @@
     <collision>
       <origin
-        xyz="0 0 0"
-        rpy="0 0 0" />
-      <geometry>
-        <mesh
-          filename="package://gummi_base_template/meshes/j7_Link.STL" />
+        xyz="0.073 0 0"
+        rpy="0 0 0" />
+      <geometry>
+        <box size=".146 .06 .015" />
       </geometry>
     </collision>
@@ -169,5 +121,5 @@
     type="revolute">
     <origin
-      xyz="0.084137 0 0.009003"
+      xyz="0.15 0 0.009003"
       rpy="0 0 0" />
     <parent
@@ -203,19 +155,21 @@
     <visual>
       <origin
-        xyz="0 0 0"
-        rpy="0 0 0" />
+        xyz="0.05 0 0"
+        rpy="0 0 0" />
+      <geometry>
+        <box size=".07 .008 .06" />
+      </geometry>
       <material
         name="">
         <color
-          rgba="0.792156862745098 0.819607843137255 0.933333333333333 1" />
+          rgba="0.79216 0.81961 0.93333 1" />
       </material>
     </visual>
     <collision>
       <origin
-        xyz="0 0 0"
-        rpy="0 0 0" />
-      <geometry>
-        <mesh
-          filename="package://gummi_base_template/meshes/gripper_Link.stl" />
+        xyz="0.05 0 0"
+        rpy="0 0 0" />
+      <geometry>
+        <box size=".07 .008 .06" />
       </geometry>
     </collision>
@@ -226,5 +180,5 @@
     type="revolute">
     <origin
-      xyz="0.066697 -0.0261 0.0093282"
+      xyz="0.14 0 0"
       rpy="1.5708 1.0472 3.1416" />
     <parent
@@ -233,5 +187,5 @@
       link="gripper_Link" />
     <axis
-      xyz="0 1 0" />
+      xyz="0 0 1" />
     <!-- <limit
       lower="-1.5708"
@@ -239,4 +193,18 @@
       effort="0"
       velocity="0" /> -->
+    <limit effort="0" lower="-2.0" upper="0.37" velocity="1.0"/>
+  </joint>
+  <link name="tool">
+  </link>
+  <joint name="coupling_tool" type="fixed">
+    <origin rpy="0 0 0" xyz="0.175 -0.02 0.13"/>
+    <parent link="wrist"/>
+    <child link="tool"/>
+    <axis xyz="0 1 0"/>
+    <!-- <limit
+    lower="-1.5708"
+    upper="1.5708"
+    effort="0"
+    velocity="0" /> -->
     <limit effort="0" lower="-0.30" upper="0.17" velocity="1.0"/>
   </joint>

File: src/gummi_ee_handshake/xacro/gummi_ee.srdf.xacro (robot description, xacro)
@@ -5,4 +5,5 @@
     <joint name="forearm_roll" />
     <joint name="wrist_pitch" />
+    <joint name="coupling_tool"/>
 </xacro:macro>
 <xacro:macro name="group_right_gripper_ee">
@@ -19,5 +20,5 @@
 <xacro:macro name="end_effector_ee">
   <!--END EFFECTOR: Purpose: Represent information about an end effector.-->
-  <end_effector name="right_eef" parent_link="wrist" group="right_gripper" />
+<end_effector group="right_arm" name="right_eef" parent_link="tool"/>
 </xacro:macro>
 <xacro:macro name="disable_collisions_ee">
@@ -25,9 +26,9 @@
   <disable_collisions link1="right_hand" link2="gripper_Link" reason="Never" /> -->
   <disable_collisions link1="gripper_Link" link2="lowerarm" reason="Never" />
-  <disable_collisions link1="gripper_Link" link2="lowerarm_preroll" reason="Never" />
+  <disable_collisions link1="gripper_Link" link2="lowerarm_preroll_d" reason="Never" />
   <disable_collisions link1="gripper_Link" link2="wrist" reason="Adjacent" />
-  <disable_collisions link1="lowerarm" link2="lowerarm_preroll" reason="Adjacent" />
+  <disable_collisions link1="lowerarm" link2="lowerarm_preroll_d" reason="Adjacent" />
   <disable_collisions link1="lowerarm" link2="wrist" reason="Adjacent" />
-  <disable_collisions link1="lowerarm_preroll" link2="wrist" reason="Never" />
+  <disable_collisions link1="lowerarm_preroll_d" link2="wrist" reason="Never" />
 </xacro:macro>
 </robot>
